Commit message: urdf

File: urdf/smarticle2.urdf (robot description, URDF)
Before this commit: robot simulation_assembly, 3 links, 2 joints
Links:
- removed link base
- removed link left_arm
- removed link right_arm
- added link arm_left, mass 0.0039735; collision mesh filename=../meshes/arm_left_visual.STL; visual mesh filename=../meshes/arm_left_visual.STL
- added link arm_right, mass 0.0039735; collision mesh filename=../meshes/arm_right.STL; visual mesh filename=../meshes/arm_right_visual.STL
- added link base_link, mass 0.033918; collision mesh filename=../meshes/base_link.STL; visual mesh filename=../meshes/base_link_visual.STL
Joints:
- removed joint left_join
- removed joint right_join
- added joint servo_left: type revolute, parent base_link, child arm_left, origin xyz=-0.0015 0.0212 0.001 rpy=0 0 0.2635, axis 0 0 -1, limit lower=-1.8 upper=1.8 effort=0.028 velocity=6.8
- added joint servo_right: type revolute, parent base_link, child arm_right, origin xyz=-0.0015 -0.0212 0.001 rpy=0 0 -1.4465, axis 0 0 -1, limit lower=-1.8 upper=1.8 effort=0.028 velocity=6.8
