Commit message: smarticle sim working

File: urdf/smarticle.urdf (robot description, URDF)
Before this commit: robot simulation_urdf, 3 links, 2 joints
Links:
- link left_arm: mass 0.00328492067362327 -> 0.00128492067362327
- link right_arm: mass 0.00328492067362327 -> 0.00128492067362327

Commit message: urdf

File: urdf/smarticle.urdf (robot description, URDF)
Before this commit: robot simulation_urdf, 3 links, 2 joints
Links:
- link base: mass 0.0461924870615736 -> 0.0339
- link left_arm: mass 0.00128492067362327 -> 0.00395
- link right_arm: mass 0.00128492067362327 -> 0.003975
Joints:
- joint left_joint: limit lower=-1.7 upper=1.7 effort=0.04 velocity=3.14 -> lower=-1.7 upper=1.7 effort=0.03 velocity=3.14
- joint right_joint: limit lower=-1.7 upper=1.7 effort=0.04 velocity=3.14 -> lower=-1.7 upper=1.7 effort=0.03 velocity=3.14

Commit message: URDF FINALLY SOLVED

File: urdf/smarticle.urdf (robot description, URDF)
Before this commit: robot simulation_urdf, 3 links, 2 joints
Links:
- removed link base
- removed link left_arm
- removed link right_arm
- added link arm_left, mass 0.0039781; collision mesh filename=../meshes/arm.STL; visual mesh filename=../meshes/arm.STL
- added link arm_right, mass 0.0039781; collision mesh filename=../meshes/arm.STL; visual mesh filename=../meshes/arm.STL
- added link base_link, mass 0.033918; collision mesh filename=../meshes/base_link.STL; visual mesh filename=../meshes/base_link.STL
Joints:
- removed joint left_joint
- removed joint right_joint
- added joint servo_left: type revolute, parent base_link, child arm_left, origin xyz=-0.0015 0.0212 0.001 rpy=0 0 1.57075, axis 0 0 1, limit lower=-1.8 upper=1.8 effort=0.03 velocity=6
- added joint servo_right: type revolute, parent base_link, child arm_right, origin xyz=-0.0015 -0.0212 0.001 rpy=0 0 -1.57075, axis 0 0 1, limit lower=-1.8 upper=1.8 effort=0.03 velocity=6

Commit message: beginning of light experiment

File: urdf/smarticle.urdf (robot description, URDF)
Before this commit: robot simulation_assembly, 3 links, 2 joints
Joints:
- joint servo_left: limit lower=-1.8 upper=1.8 effort=0.03 velocity=6 -> lower=-1.8 upper=1.8 effort=0.025 velocity=6
- joint servo_right: limit lower=-1.8 upper=1.8 effort=0.03 velocity=6 -> lower=-1.8 upper=1.8 effort=0.025 velocity=6

Commit message: add friction value to urdf and change old arms

File: urdf/smarticle.urdf (robot description, URDF)
Before this commit: robot simulation_assembly, 3 links, 2 joints
Links:
- link arm_left: geometry collision mesh filename=../meshes/arm.STL; visual mesh filename=../meshes/arm.STL
- link arm_right: geometry collision mesh filename=../meshes/arm.STL; visual mesh filename=../meshes/arm.STL

Commit message: ray arms

File: urdf/smarticle.urdf (robot description, URDF)
Before this commit: robot simulation_assembly, 3 links, 2 joints
Links:
- link arm_left: geometry collision mesh filename=../meshes/ray_arm.STL; visual mesh filename=../meshes/ray_arm.STL
- link arm_right: geometry collision mesh filename=../meshes/ray_arm.STL; visual mesh filename=../meshes/ray_arm.STL
