Commit message: ring stuff

File: urdf/ring.urdf (robot description, URDF)
Before this commit: robot part1, 1 links, 0 joints
Links:
- link ring: geometry collision mesh filename=../meshes/tall_ring.obj; visual mesh filename=../meshes/tall_ring.obj

Commit message: ring_good

File: urdf/ring.urdf (robot description, URDF)
Before this commit: robot part1, 1 links, 0 joints
Links:
- link ring: geometry collision mesh filename=../meshes/tall_ring2.obj; visual mesh filename=../meshes/ring.STL

Commit message: update urdfs

File: urdf/ring.urdf (robot description, URDF)
Before this commit: robot part1, 1 links, 0 joints
Links:
- link ring: geometry collision mesh filename=../meshes/20mm_ring.obj; visual mesh filename=../meshes/20mm_ring.STL

File: urdf/smarticle.urdf (robot description, URDF)
Before this commit: robot simulation_assembly, 3 links, 2 joints
Links:
- link arm_left: geometry collision mesh filename=../meshes/ray_arm.STL; visual mesh filename=../meshes/ray_arm.STL
- link arm_right: geometry collision mesh filename=../meshes/ray_arm.STL; visual mesh filename=../meshes/ray_arm.STL

Commit message: playing with friction

File: urdf/ring.urdf (robot description, URDF)
Before this commit: robot part1, 1 links, 0 joints
Links:
- link ring: geometry collision mesh filename=../meshes/20mm_ring.obj scale=1 1 1; visual mesh filename=../meshes/20mm_ring.STL scale=1 1 1

File: urdf/smarticle.urdf (robot description, URDF)
Before this commit: robot simulation_assembly, 3 links, 2 joints
Joints:
- joint servo_left: limit lower=-1.8 upper=1.8 effort=0.025 velocity=6 -> lower=-1.8 upper=1.8 effort=0.01 velocity=6
- joint servo_right: limit lower=-1.8 upper=1.8 effort=0.025 velocity=6 -> lower=-1.8 upper=1.8 effort=0.01 velocity=6

Commit message: created new cornell branch and updated urdf/run file

File: urdf/ring.urdf (robot description, URDF)
Before this commit: robot part1, 1 links, 0 joints
Links:
- link ring: geometry collision mesh filename=../meshes/20mm_ring.obj scale=10 10 20; visual mesh filename=../meshes/20mm_ring.STL scale=10 10 20
