Commit message: new urdf

File: simulation_assembly/urdf/simulation_assembly.urdf (robot description, URDF)
Before this commit: robot sim_urdf, 3 links, 2 joints
Links:
- link arm_left: mass 0.0039781 -> 0.0039735; geometry collision mesh filename=package://simulation_assembly/meshes/arm_left.STL; visual mesh filename=package://simulation_assembly/meshes/arm_left.STL
- link arm_right: mass 0.0039781 -> 0.0039735; geometry collision mesh filename=package://simulation_assembly/meshes/arm_right.STL; visual mesh filename=package://simulation_assembly/meshes/arm_right.STL
- link base_link: geometry collision mesh filename=package://simulation_assembly/meshes/base_link.STL; visual mesh filename=package://simulation_assembly/meshes/base_link.STL
Joints:
- removed joint servo_right
- added joint servo_rigth: type revolute, parent base_link, child arm_right, origin xyz=-0.0015 -0.0212 0.001 rpy=0 0 0, axis 0 0 1, limit lower=-1.8 upper=1.8 effort=0.03 velocity=6
- joint servo_left: limit lower=-1.8 upper=1.8 effort=0.03 velocity=6 -> (none); origin xyz=-0.0015 -0.001 0.0212 rpy=1.5708 0 0 -> xyz=-0.0015 0.0212 0.001 rpy=0 0 0; type revolute -> continuous
